Commit message: create tugbot_gazebo pkg

File: tugbot_description/urdf/model.urdf (robot description, URDF)
Before this commit: robot tugbot, 10 links, 9 joints
Links:
- removed link scan_back
- removed link scan_front
- added link tugbot/scan_back/scan_back
- added link tugbot/scan_front/scan_front
Joints:
- joint scan_back_joint: child scan_back -> tugbot/scan_back/scan_back
- joint scan_front_joint: child scan_front -> tugbot/scan_front/scan_front

Commit message: use 3d lidar for slam-toolbox

File: tugbot_description/urdf/model.urdf (robot description, URDF)
Before this commit: robot tugbot, 10 links, 9 joints
Links:
- removed link scan_omni
- added link tugbot/scan_omni/scan_omni; visual cylinder length=0.0015 radius=0.06; visual cylinder length=0.09 radius=0.005
Joints:
- joint scan_omni_joint: child scan_omni -> tugbot/scan_omni/scan_omni
